File: Tof_PCB.sch (KiCad schematic (older format))
At the start: 96 parts, among them J1 Screw_Terminal_01x02, J2 Screw_Terminal_01x02, J3 Screw_Terminal_01x02, J4 Conn_02x03_Odd_Even, J5 Conn_01x04, J6 Conn_01x04, J7 Screw_Terminal_01x02, SW1 SW_Push, U1 ATmega328PB-MU, U2 DAC128S085, U3 LM4132BMF, U31 LM321, U33 UMCC_50Ohm, Y1 Crystal_GND24

Commit message: changed 100k resistor and tlv3501 digikey numbers
Parts:
- R75: Digi-Key_PN RMCF0603FT110K -> P100KDATR-ND
Changed lines of the file:
@@
 F 2 "Resistor_SMD:R_0603_1608Metric" V 7930 4500 50  0001 C CNN
 F 3 "~" H 8000 4500 50  0001 C CNN
-F 4 "RMCF0603FT110K" H 8000 4500 50  0001 C CNN "Digi-Key_PN"
+F 4 "P100KDATR-ND" H 8000 4500 50  0001 C CNN "Digi-Key_PN"
 	1    8000 4500
 	0    1    1    0
