File: Tof_Rx.sch (KiCad schematic (older format))
At the start: 82 parts, among them IC1 NC7WZ00K8X, M3 mounting_holes_laser, M4 mounting_holes_laser, U15 LMH6559MF, U16 SiPM-MicroRB, U17 UMCC_50Ohm, U18 ts5a4596, U19 ts5a4596, U20 MAX40658, U21 LP5907MFX-3.3_NOPB, U22 UMCC_50Ohm, U23 TLV3501, U24 TLV3501, U25 HMC589AST89E, U26 UMCC_50Ohm, U27 UMCC_50Ohm, U28 UMCC_50Ohm, U29 UMCC_50Ohm

Commit message: Added RLC values
Parts:
- removed C42, C43: C, Capacitor_SMD:C_0603_1608Metric, symbol Device:C
- removed R65, R71: R, Resistor_SMD:R_0603_1608Metric, symbol Device:R
- removed U26: UMCC_50Ohm, IODA_Lib:Molex_734120114_UMC_RF_CONN_Vertical, symbol ioda:UMCC_50Ohm
- added C57, C68, C70, C71: 2.2uF, Capacitor_SMD:C_0603_1608Metric, symbol Device:C
- added C58, C62, C63, C64, C69, C72: 100nF, Capacitor_SMD:C_0603_1608Metric, symbol Device:C
- added L20: L, Inductor_SMD:L_0603_1608Metric, symbol Device:L
- added L21: 10uH, Inductor_SMD:L_0603_1608Metric, symbol Device:L
- added R14, R78, R79: 200R, Resistor_SMD:R_0603_1608Metric, symbol Device:R
- added R76, R77: 50k, Resistor_SMD:R_0603_1608Metric, symbol Device:R
- added TP10, TP9: TestPoint, Connector_PinHeader_1.00mm:PinHeader_1x01_P1.00mm_Vertical, symbol Connector:TestPoint
- added unit 2 of U26
- added unit 3 of U30
- added unit 2 of U30
- added U32: UMCC_50Ohm, IODA_Lib:Molex_734120114_UMC_RF_CONN_Vertical, symbol ioda:UMCC_50Ohm
- C27, C31, C32, C33, C35, C36, C37, C38, C39, C41, C44, C48, C49, C50, C52, C54: value C -> 2.2uF
- C28, C29, C30, C40, C45, C46, C47, C51, C53: value C -> 100nF
- C34: value C -> 1uF
- L18, L19: value L -> 10uH
- R50, R67: value R -> 0R
- R51: value R -> 1M
- R52, R53, R70: value R -> 50R
- R54, R56, R57, R58, R60, R68, R69: value R -> 10k
- R55, R61, R72: value R -> 200R
- R59, R63: value R -> 75R
- R62: value R -> 100k
- R64: value R -> 150R
- R66: value R -> 1.8R
- renumbered IC1 to U26, IC1 to U30
Connections:
- wire segments 110 -> 135
- no-connect marks 0 -> 2
Other:
- note added: "Bias-T for RF-amp"
- note added: "Biasing"
- moved on the sheet: C28, C29, C33, C34, C37, C38, C46, C47, C48, C49, C50, C51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

Commit message: Added more digikey numbers in BOM
Parts:
- C27: value 2.2uF -> 10nF, 250V
- C28, C29: value 100nF -> 10nF, 250V
- D3: symbol ioda:MTAPD-06 -> ioda:MTAPD-06-013; Digi-Key_PN (none) -> 1125-1298-ND
- D4: Digi-Key_PN (none) -> BAS170WS-E3-08GICT-ND
- L12, L13, L14, L15, L16, L17, L20: Digi-Key_PN (none) -> 490-5216-1-ND
- TP10, TP4, TP5, TP6, TP9: Digi-Key_PN (none) -> 732-5314-ND
- U15: Digi-Key_PN (none) -> 296-46123-1-ND
- U16: Digi-Key_PN (none) -> MICRORB-10020-MLP-TR1OS-ND
- U17, U22, U27, U28, U29, U32: Digi-Key_PN (none) -> A118077CT-ND
- U18, U19: Digi-Key_PN (none) -> 296-17709-1-ND
- U20: value MAX40658 -> MAX40659; symbol ioda:MAX40658 -> ioda:MAX40659; Digi-Key_PN (none) -> MAX40659ETA+TCT-ND; Field5 MAX40658ETA+-ND -> MAX40659ETA+-ND
- U21: Digi-Key_PN (none) -> 296-38557-1-ND
- U23, U24: Digi-Key_PN (none) -> 296-43611-1-ND
- U25: Digi-Key_PN (none) -> 1127-3329-1-ND
- U26, U30: Digi-Key_PN (none) -> NC7WZ00K8XCT-ND
Connections:
- wire segments 135 -> 141
- no-connect marks 2 -> 3
Other:
- moved on the sheet: M4, U26B

Commit message: solved drc errors
Connections:
- net buffer_out: now reaches R14.1, R52.2, U15.1 (OUT), U18.2 (COM), U19.2 (COM)
Changed lines of the file:
@@
-$EndComp
-$Comp
-L power:GND #PWR?
-U 1 1 5DDE9A1C
-P 8650 5000
-AR Path="/5DDE9A1C" Ref="#PWR?"  Part="1"
-AR Path="/5DB7F50A/5DDE9A1C" Ref="#PWR?"  Part="1"
-AR Path="/5DD4CF74/5DDE9A1C" Ref="#PWR0125"  Part="1"
-F 0 "#PWR0125" H 8650 4750 50  0001 C CNN
-F 1 "GND" H 8655 4827 50  0000 C CNN
-F 2 "" H 8650 5000 50  0001 C CNN
-F 3 "" H 8650 5000 50  0001 C CNN
-	1    8650 5000
-	1    0    0    -1
 $EndComp
 $Comp
@@
 Wire Wire Line
 	1700 3900 1600 3900
+Text Label 2600 5850 0    50   ~ 0
+buffer_out
+$Comp
+L power:GND #PWR?
+U 1 1 5E49E4FE
+P 8650 5000
+AR Path="/5E49E4FE" Ref="#PWR?"  Part="1"
+AR Path="/5DB7F50A/5E49E4FE" Ref="#PWR?"  Part="1"
+AR Path="/5DD4CF74/5E49E4FE" Ref="#PWR0125"  Part="1"
+F 0 "#PWR0125" H 8650 4750 50  0001 C CNN
+F 1 "GND" H 8655 4827 50  0000 C CNN
+F 2 "" H 8650 5000 50  0001 C CNN
+F 3 "" H 8650 5000 50  0001 C CNN
+	1    8650 5000
+	1    0    0    -1
+$EndComp
 $EndSCHEMATC

Commit message: bugfixes
Parts:
- added C77: c_rf_filt, Capacitor_SMD:C_0603_1608Metric, symbol Device:C
- added C81: 2.2uF, Capacitor_SMD:C_0603_1608Metric, symbol Device:C
- added R88: 0R, Resistor_SMD:R_0603_1608Metric, symbol Device:R
- added R89, R90, R91: 22R, Resistor_SMD:R_0603_1608Metric, symbol Device:R
- added U35: UMCC_50Ohm, IODA_Lib:Molex_734120114_UMC_RF_CONN_Vertical, symbol ioda:UMCC_50Ohm
- C27, C28, C29: Digi-Key_PN (none) -> 732-12168-1-ND
- C30, C40, C45, C46, C47, C51, C53, C58, C62, C63, C64, C69, C72: Digi-Key_PN (none) -> 490-3285-1-ND
- C31, C32, C33, C35, C36, C37, C38, C39, C41, C44, C48, C49, C50, C52, C54, C57, C68, C70, C71: Digi-Key_PN (none) -> 490-12740-1-ND
- C34: value 1uF -> 2.2uF; Digi-Key_PN (none) -> 490-12740-1-ND
- D3, U16: Configuration (none) -> do not mount
- L12, L13, L14, L15, L16, L17, L20: value L -> bead
- L18, L19, L21: Digi-Key_PN (none) -> 490-4025-1-ND
- R14, R55, R61, R72, R78, R79: Digi-Key_PN (none) -> RHM200ADCT-ND
- R50, R67: Configuration (none) -> do not mount; Digi-Key_PN (none) -> RMCF0603ZT0R00CT-ND
- R51: Digi-Key_PN (none) -> 311-1.00MHRCT-ND
- R52, R53, R70: Digi-Key_PN (none) -> 541-56.0SCT-ND; Field4 (none) -> P49.9HCT-ND
- R54, R56, R57, R58, R60, R68, R69: Digi-Key_PN (none) -> P10.0KHCT-ND
- R59: Digi-Key_PN (none) -> RNCP0603FTD75R0CT-ND
- R62: Digi-Key_PN (none) -> RMCF0603FT110K
- R63: Configuration (none) -> do not mount; Digi-Key_PN (none) -> RNCP0603FTD75R0CT-ND
- R64: value 150R -> 22R; Digi-Key_PN (none) -> A129668CT-ND
- R66: Digi-Key_PN (none) -> 541-1.80CCCT-ND
- R76, R77: value 50k -> 100k; Digi-Key_PN (none) -> RMCF0603FT110K
Connections:
- net +5V: no longer U30.5 (A2), U30.6 (B2)
- net GND: now also C77.2, U35.1, U35.3; no longer R64.2
- net TIA_out: now also R67.2, R88.2; no longer C37.2
- net rfamp_out: now also C77.1, C81.2; no longer R70.2, R72.1
- net at C70.2, U25.1: no longer R67.2
- net at U27.2: now also R90.1; no longer U30.7 (Y1)
- net at U28.2: now also R91.1; no longer U26.7 (Y1)
- net con: now reaches C38.2, R59.1, R61.2
- net con: now also R88.1; no longer R63.1
- net at U30.3 (Y2): now also R89.2
- new net: C37.2, R63.1, R64.2
- new net: R90.2, U30.5 (A2), U30.6 (B2), U30.7 (Y1)
- new net: R91.2, U26.7 (Y1)
- new net: C81.1, R70.2, R72.1
- new net: R89.1, U35.2
- no-connect marks 3 -> 1
Other:
- note added: "APD"
- note added: "Comparator"
- note added: "Lock-in Amp"
- note added: "RF-Amp"
- note added: "SiPM"
- note added: "optional filtering"
- moved on the sheet: C46, C49, C53, C57, C58, L16, L20, R59, R64, R67, R70, U27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

Commit message: changed 100k resistor and tlv3501 digikey numbers
Parts:
- R62, R76, R77: Digi-Key_PN RMCF0603FT110K -> P100KDATR-ND
- U23, U24: Digi-Key_PN 296-43611-1-ND -> 296-35977-1-ND
Changed lines of the file:
@@
 F 2 "IODA_Lib:SOT-23-6" H 8150 3800 50  0001 C CNN
 F 3 "https://www.ti.com/lit/ds/symlink/tlv3501.pdf" H 8150 3800 50  0001 C CNN
-F 4 "296-43611-1-ND" H 0   0   50  0001 C CNN "Digi-Key_PN"
+F 4 "296-35977-1-ND" H 0   0   50  0001 C CNN "Digi-Key_PN"
 	1    8150 3800
 	1    0    0    -1
@@
 F 2 "IODA_Lib:SOT-23-6" H 8150 5300 50  0001 C CNN
 F 3 "https://www.ti.com/lit/ds/symlink/tlv3501.pdf" H 8150 5300 50  0001 C CNN
-F 4 "296-43611-1-ND" H 0   0   50  0001 C CNN "Digi-Key_PN"
+F 4 "296-35977-1-ND" H 0   0   50  0001 C CNN "Digi-Key_PN"
 	1    8150 5300
 	1    0    0    -1
@@
 F 2 "Resistor_SMD:R_0603_1608Metric" V 5630 6550 50  0001 C CNN
 F 3 "~" H 5700 6550 50  0001 C CNN
-F 4 "RMCF0603FT110K" H 5700 6550 50  0001 C CNN "Digi-Key_PN"
+F 4 "P100KDATR-ND" H 5700 6550 50  0001 C CNN "Digi-Key_PN"
 	1    5700 6550
 	-1   0    0    1
@@
 F 2 "Resistor_SMD:R_0603_1608Metric" V 7230 3950 50  0001 C CNN
 F 3 "~" H 7300 3950 50  0001 C CNN
-F 4 "RMCF0603FT110K" H 7300 3950 50  0001 C CNN "Digi-Key_PN"
+F 4 "P100KDATR-ND" H 7300 3950 50  0001 C CNN "Digi-Key_PN"
 	1    7300 3950
 	0    1    1    0
@@
 F 2 "Resistor_SMD:R_0603_1608Metric" V 7230 5450 50  0001 C CNN
 F 3 "~" H 7300 5450 50  0001 C CNN
-F 4 "RMCF0603FT110K" H 7300 5450 50  0001 C CNN "Digi-Key_PN"
+F 4 "P100KDATR-ND" H 7300 5450 50  0001 C CNN "Digi-Key_PN"
 	1    7300 5450
 	0    1    1    0
